File: cpu.kicad_sch (KiCad schematic)
At the start: 19 parts, among them U1 Intel_8088, U11 74HCT373, U14 SN74HCT245N, U2 8087, U3 8284, U6 8288, Y1 14.31818 MHz

Commit message: Fix ERC errors
Signed-off-by: Lucy Mielke <user@domain.tld>
Connections:
- net a10 renamed addr10
- net a11 renamed addr11
- net a12 renamed addr12
- net a13 renamed addr13
- net a14 renamed addr14
- net a15 renamed addr15
- net a16 renamed addr16
- net a17 renamed addr17
- net a18 renamed addr18
- net a19 renamed addr19
- net a8 renamed addr8
- net a9 renamed addr9
- no-connect marks 0 -> 12
Other:
- moved on the sheet: C13, C16, U11, U14
