File: io_ethernet.kicad_sch (KiCad schematic)
At the start: 10 parts, among them J6 RJ45_Amphenol_RJMG1BD3B8K1ANR, U26 Realtek RTL8019AS, U27 93LCxxC

Commit message: Fix ERC errors
Signed-off-by: Lucy Mielke <user@domain.tld>
Connections:
- no-connect marks 10 -> 36
Changed lines of the file:
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@@
+	)
+	(no_connect
+		(at 97.79 50.8)
 	)
 	(no_connect
@@
 	)
 	(no_connect
+		(at 97.79 127)
+	)
+	(no_connect
+		(at 97.79 132.08)
+	)
+	(no_connect
+		(at 57.15 175.26)
+	)
+	(no_connect
 		(at 57.15 111.76)
 	)
 	(no_connect
+		(at 97.79 106.68)
+	)
+	(no_connect
+		(at 97.79 45.72)
+	)
+	(no_connect
+		(at 97.79 86.36)
+	)
+	(no_connect
 		(at 97.79 179.07)
 	)
 	(no_connect
+		(at 97.79 66.04)
+	)
+	(no_connect
+		(at 97.79 109.22)
+	)
+	(no_connect
 		(at 97.79 173.99)
 	)
 	(no_connect
+		(at 97.79 99.06)
+	)
+	(no_connect
+		(at 97.79 43.18)
+	)
+	(no_connect
+		(at 97.79 124.46)
+	)
+	(no_connect
+		(at 97.79 101.6)
+	)
+	(no_connect
+		(at 97.79 137.16)
+	)
+	(no_connect
+		(at 97.79 129.54)
+	)
+	(no_connect
+		(at 97.79 93.98)
+	)
+	(no_connect
+		(at 57.15 170.18)
+	)
+	(no_connect
 		(at 97.79 176.53)
 	)
 	(no_connect
+		(at 97.79 76.2)
+	)
+	(no_connect
+		(at 97.79 91.44)
+	)
+	(no_connect
+		(at 97.79 104.14)
+	)
+	(no_connect
+		(at 57.15 167.64)
+	)
+	(no_connect
+		(at 97.79 134.62)
+	)
+	(no_connect
+		(at 97.79 53.34)
+	)
+	(no_connect
+		(at 97.79 38.1)
+	)
+	(no_connect
+		(at 97.79 81.28)
+	)
+	(no_connect
 		(at 57.15 40.64)
+	)
+	(no_connect
+		(at 97.79 96.52)
 	)
 	(no_connect
@@
 		)
 	)
-	(hierarchical_label "{DATA_BUS}"
+	(hierarchical_label "d[0..7]"
 		(shape bidirectional)
 		(at 48.26 158.75 180)
@@
 		)
 	)
-	(hierarchical_label "{ADDRESS_BUS}"
+	(hierarchical_label "addr[0..19]"
 		(shape bidirectional)
 		(at 45.72 46.99 180)
