File: io_ide.kicad_sch (KiCad schematic)
At the start: 13 parts, among them J7 Conn_02x20_Odd_Even, U28 74HCT688 (CD74HCT688E), U29 SN74HCT245N, U30 SN74HCT245N, U31 SN74HCT573N, U32 SN74HCT32N

Commit message: Fix ERC errors
Signed-off-by: Lucy Mielke <user@domain.tld>
Connections:
- no-connect marks 8 -> 11
Changed lines of the file:
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@@
+	)
+	(no_connect
+		(at 29.21 172.72)
+	)
+	(no_connect
+		(at 29.21 175.26)
 	)
 	(no_connect
@@
 	(no_connect
 		(at 227.33 93.98)
+	)
+	(no_connect
+		(at 64.77 165.1)
 	)
 	(no_connect
@@
 		)
 	)
-	(hierarchical_label "{IDE_BUS}"
+	(hierarchical_label "IDE_D[0..15]"
 		(shape bidirectional)
 		(at 233.68 46.99 90)
@@
 		)
 	)
-	(hierarchical_label "{ADDRESS_BUS}"
+	(hierarchical_label "addr[0..19]"
 		(shape bidirectional)
 		(at 21.59 146.05 0)
@@
 		)
 	)
-	(hierarchical_label "{DATA_BUS}"
+	(hierarchical_label "d[0..7]"
 		(shape bidirectional)
 		(at 194.31 142.24 0)
@@
 		)
 	)
-	(hierarchical_label "{ADDRESS_BUS}"
+	(hierarchical_label "addr[0..19]"
 		(shape bidirectional)
 		(at 218.44 78.74 180)
@@
 		)
 	)
-	(hierarchical_label "{DATA_BUS}"
+	(hierarchical_label "d[0..7]"
 		(shape bidirectional)
 		(at 63.5 137.16 180)
@@
 		)
 	)
-	(hierarchical_label "{ADDRESS_BUS}"
+	(hierarchical_label "addr[0..19]"
 		(shape bidirectional)
 		(at 29.21 43.18 180)
@@
 		)
 	)
-	(hierarchical_label "{IDE_BUS}"
+	(hierarchical_label "IDE_D[0..15]"
 		(shape bidirectional)
 		(at 133.35 138.43 180)
