File: io_isa.kicad_sch (KiCad schematic)
At the start: 7 parts, among them J10 Bus_ISA_8bit, J8 Bus_ISA_8bit, J9 Bus_ISA_8bit, U33 L7905

Commit message: Fix ERC errors
Signed-off-by: Lucy Mielke <user@domain.tld>
Connections:
- no-connect marks 5 -> 51
Changed lines of the file:
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@@
 	)
 	(no_connect
+		(at 124.46 90.17)
+	)
+	(no_connect
+		(at 245.11 80.01)
+	)
+	(no_connect
 		(at 124.46 72.39)
 	)
 	(no_connect
+		(at 124.46 92.71)
+	)
+	(no_connect
+		(at 209.55 110.49)
+	)
+	(no_connect
+		(at 46.99 100.33)
+	)
+	(no_connect
+		(at 124.46 115.57)
+	)
+	(no_connect
+		(at 124.46 120.65)
+	)
+	(no_connect
+		(at 209.55 115.57)
+	)
+	(no_connect
+		(at 46.99 115.57)
+	)
+	(no_connect
+		(at 209.55 113.03)
+	)
+	(no_connect
+		(at 46.99 92.71)
+	)
+	(no_connect
 		(at 82.55 80.01)
 	)
 	(no_connect
+		(at 209.55 97.79)
+	)
+	(no_connect
+		(at 46.99 113.03)
+	)
+	(no_connect
+		(at 209.55 92.71)
+	)
+	(no_connect
+		(at 209.55 67.31)
+	)
+	(no_connect
+		(at 209.55 90.17)
+	)
+	(no_connect
+		(at 124.46 100.33)
+	)
+	(no_connect
+		(at 46.99 67.31)
+	)
+	(no_connect
+		(at 209.55 95.25)
+	)
+	(no_connect
+		(at 46.99 97.79)
+	)
+	(no_connect
+		(at 124.46 113.03)
+	)
+	(no_connect
 		(at 209.55 72.39)
 	)
 	(no_connect
+		(at 245.11 54.61)
+	)
+	(no_connect
+		(at 124.46 67.31)
+	)
+	(no_connect
+		(at 209.55 118.11)
+	)
+	(no_connect
+		(at 245.11 77.47)
+	)
+	(no_connect
+		(at 209.55 107.95)
+	)
+	(no_connect
+		(at 160.02 80.01)
+	)
+	(no_connect
+		(at 46.99 107.95)
+	)
+	(no_connect
+		(at 46.99 118.11)
+	)
+	(no_connect
+		(at 160.02 77.47)
+	)
+	(no_connect
 		(at 46.99 72.39)
 	)
@@
 		(at 82.55 77.47)
 	)
+	(no_connect
+		(at 124.46 95.25)
+	)
+	(no_connect
+		(at 209.55 62.23)
+	)
+	(no_connect
+		(at 209.55 120.65)
+	)
+	(no_connect
+		(at 160.02 54.61)
+	)
+	(no_connect
+		(at 209.55 100.33)
+	)
+	(no_connect
+		(at 46.99 95.25)
+	)
+	(no_connect
+		(at 124.46 118.11)
+	)
+	(no_connect
+		(at 82.55 54.61)
+	)
+	(no_connect
+		(at 124.46 62.23)
+	)
+	(no_connect
+		(at 124.46 97.79)
+	)
+	(no_connect
+		(at 46.99 120.65)
+	)
+	(no_connect
+		(at 46.99 105.41)
+	)
+	(no_connect
+		(at 124.46 105.41)
+	)
+	(no_connect
+		(at 124.46 107.95)
+	)
+	(no_connect
+		(at 46.99 90.17)
+	)
+	(no_connect
+		(at 46.99 110.49)
+	)
 	(bus_entry
 		(at 90.17 64.77)
@@
 		)
 	)
-	(hierarchical_label "{DATA_BUS}"
+	(hierarchical_label "d[0..7]"
 		(shape bidirectional)
 		(at 170.18 80.01 0)
@@
 		)
 	)
-	(hierarchical_label "{DATA_BUS}"
+	(hierarchical_label "d[0..7]"
 		(shape bidirectional)
 		(at 255.27 80.01 0)
@@
 		)
 	)
-	(hierarchical_label "{ADDRESS_BUS}"
+	(hierarchical_label "addr[0..19]"
 		(shape bidirectional)
 		(at 255.27 142.24 270)
@@
 		)
 	)
-	(hierarchical_label "{ADDRESS_BUS}"
+	(hierarchical_label "addr[0..19]"
 		(shape bidirectional)
 		(at 170.18 142.24 270)
@@
 		)
 	)
-	(hierarchical_label "{ADDRESS_BUS}"
+	(hierarchical_label "addr[0..19]"
 		(shape bidirectional)
 		(at 92.71 142.24 270)
@@
 		)
 	)
-	(hierarchical_label "{DATA_BUS}"
+	(hierarchical_label "d[0..7]"
 		(shape bidirectional)
 		(at 92.71 80.01 0)
@@
 	)
 	(symbol
+		(lib_name "Bus_ISA_8bit_1")
 		(lib_id "Connector:Bus_ISA_8bit")
 		(at 64.77 92.71 0)
@@
 	)
 	(symbol
+		(lib_name "Bus_ISA_8bit_2")
 		(lib_id "Connector:Bus_ISA_8bit")
 		(at 142.24 92.71 0)
