File: io_pit.kicad_sch (KiCad schematic)
At the start: 4 parts, among them U24 8254

Commit message: Fix ERC errors
Signed-off-by: Lucy Mielke <user@domain.tld>
Changed lines of the file:
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@@
 		)
 	)
-	(hierarchical_label "{ADDRESS_BUS}"
+	(hierarchical_label "addr[0..19]"
 		(shape bidirectional)
 		(at 118.11 83.82 180)
@@
 		)
 	)
-	(hierarchical_label "{DATA_BUS}"
+	(hierarchical_label "d[0..7]"
 		(shape bidirectional)
 		(at 121.92 41.91 180)
