File: io_rs232_uart.kicad_sch (KiCad schematic)
At the start: 23 parts, among them J3 DE-9SA-J4-2R, U19 TL16C550BN, U20 CD74HCT30E, U21 MAX232, U22 MAX232, Y2 1.8432MHZ

Commit message: add PIT
Signed-off-by: Lucy Mielke <user@domain.tld>
Changed lines of the file:
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@@
-		)
-	)
-	(label "UART_IRQ"
-		(at 58.42 147.32 180)
-		(effects
-			(font
-				(size 1.27 1.27)
-			)
-			(justify right bottom)
 		)
 	)
@@
 		(effects
 			(font
+				(size 1.27 1.27)
+			)
+			(justify right)
+		)
+	)
+	(hierarchical_label "UART_IRQ"
+		(shape output)
+		(at 58.42 147.32 180)
+		(effects
+			(font

Commit message: Fix ERC errors
Signed-off-by: Lucy Mielke <user@domain.tld>
Connections:
- no-connect marks 2 -> 10
Changed lines of the file:
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@@
+	)
+	(no_connect
+		(at 109.22 132.08)
 	)
 	(no_connect
@@
 	)
 	(no_connect
+		(at 109.22 106.68)
+	)
+	(no_connect
+		(at 109.22 144.78)
+	)
+	(no_connect
+		(at 58.42 144.78)
+	)
+	(no_connect
 		(at 209.55 73.66)
+	)
+	(no_connect
+		(at 109.22 99.06)
+	)
+	(no_connect
+		(at 109.22 129.54)
+	)
+	(no_connect
+		(at 109.22 149.86)
+	)
+	(no_connect
+		(at 109.22 134.62)
 	)
 	(bus_entry
@@
 		)
 	)
-	(hierarchical_label "{ADDRESS_BUS}"
+	(hierarchical_label "addr[0..19]"
 		(shape bidirectional)
 		(at 30.48 55.88 0)
@@
 		)
 	)
-	(hierarchical_label "{ADDRESS_BUS}"
+	(hierarchical_label "addr[0..19]"
 		(shape bidirectional)
 		(at 49.53 109.22 180)
@@
 		)
 	)
-	(hierarchical_label "{DATA_BUS}"
+	(hierarchical_label "d[0..7]"
 		(shape bidirectional)
 		(at 53.34 99.06 180)
