File: memory.kicad_sch (KiCad schematic)
At the start: 17 parts, among them U10 AS6C4008-55PCN, U15 AS6C4008-55PCN, U16 28C256, U17 CD74HCT14E, U18 CD74HCT10E, U7 SN74HCT138N, U8 SN74HCT08N, U9 CD74HCT21E

Commit message: Complete UART connection
Signed-off-by: Lucy Mielke <user@domain.tld>
Connections:
- net RSTBTN: now reaches U17.3 (2A)
- net RSTBTN_INV: now reaches U17.4 (2Y)
Changed lines of the file:
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@@
+		)
+	)
+	(wire
+		(pts
+			(xy 170.18 68.58) (xy 175.26 68.58)
+		)
+		(stroke
+			(width 0)
+			(type default)
 		)
 	)
@@
 		(pts
 			(xy 77.47 24.13) (xy 77.47 48.26)
+		)
+		(stroke
+			(width 0)
+			(type default)
+		)
+	)
+	(wire
+		(pts
+			(xy 170.18 71.12) (xy 175.26 71.12)
 		)
 		(stroke
@@
 			)
 			(justify left bottom)
+		)
+	)
+	(hierarchical_label "RSTBTN_INV"
+		(shape output)
+		(at 170.18 71.12 180)
+		(effects
+			(font
+				(size 1.27 1.27)
+			)
+			(justify right)
 		)
 	)
@@
 		)
 	)
+	(hierarchical_label "RSTBTN"
+		(shape input)
+		(at 170.18 68.58 180)
+		(effects
+			(font
+				(size 1.27 1.27)
+			)
+			(justify right)
+		)
+	)

Commit message: reorganise
Signed-off-by: Lucy Mielke <user@domain.tld>
Other:
- note added: "Memory (RAM/ROM)"
Changed lines of the file:
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@@
 		(comment 1 "${COMMENT1}")
+	)
+	(text "Memory (RAM/ROM)"
+		(exclude_from_sim no)
+		(at 148.59 16.51 0)
+		(effects
+			(font
+				(size 1.905 1.905)
+			)
+		)
 	)
 	(junction

Commit message: IDE controller/connector
Signed-off-by: Lucy Mielke <user@domain.tld>
Connections:
- net addr0: now also U17.5 (3A)
- net IO_ACT: now reaches U7.4 (~{G2A}), U8.3 (1Y)
- net addr0_INV: now reaches U17.6 (3Y)
Changed lines of the file:
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@@
+	)
+	(bus_entry
+		(at 168.91 73.66)
+		(size -2.54 2.54)
+		(stroke
+			(width 0)
+			(type default)
+		)
 	)
 	(bus_entry
@@
 	(bus
 		(pts
-			(xy 180.34 100.33) (xy 180.34 147.32)
+			(xy 180.34 88.9) (xy 180.34 147.32)
 		)
 		(stroke
@@
 	(wire
 		(pts
+			(xy 168.91 73.66) (xy 175.26 73.66)
+		)
+		(stroke
+			(width 0)
+			(type default)
+		)
+	)
+	(wire
+		(pts
 			(xy 137.16 45.72) (xy 137.16 40.64)
 		)
@@
 		)
 	)
+	(bus
+		(pts
+			(xy 166.37 76.2) (xy 166.37 88.9)
+		)
+		(stroke
+			(width 0)
+			(type default)
+		)
+	)
 	(wire
 		(pts
@@
 		)
 	)
+	(bus
+		(pts
+			(xy 180.34 88.9) (xy 166.37 88.9)
+		)
+		(stroke
+			(width 0)
+			(type default)
+		)
+	)
 	(wire
 		(pts
@@
 		(pts
 			(xy 77.47 146.05) (xy 77.47 161.29)
-		)
-		(stroke
-			(width 0)
-			(type default)
-		)
-	)
-	(wire
-		(pts
-			(xy 60.96 40.64) (xy 85.09 40.64)
 		)
 		(stroke
@@
 	(label "addr19"
 		(at 80.01 50.8 0)
+		(effects
+			(font
+				(size 1.27 1.27)
+			)
+			(justify left bottom)
+		)
+	)
+	(label "addr0"
+		(at 168.91 73.66 0)
 		(effects
 			(font
@@
 		)
 	)
+	(hierarchical_label "IO_ACT"
+		(shape input)
+		(at 85.09 40.64 180)
+		(effects
+			(font
+				(size 1.27 1.27)
+			)
+			(justify right)
+		)
+	)
 	(hierarchical_label "MRDC"
 		(shape input)
@@
 		)
 	)
+	(hierarchical_label "IO_ACT"
+		(shape input)
+		(at 60.96 40.64 0)
+		(effects
+			(font
+				(size 1.27 1.27)
+			)
+			(justify left)
+		)
+	)
 	(hierarchical_label "MRDC"
 		(shape input)
@@
 		)
 	)
+	(hierarchical_label "addr0_INV"
+		(shape output)
+		(at 175.26 76.2 180)
+		(effects
+			(font
+				(size 1.27 1.27)
+			)
+			(justify right)
+		)
+	)

Commit message: Fix ERC errors
Signed-off-by: Lucy Mielke <user@domain.tld>
Connections:
- no-connect marks 10 -> 31
Changed lines of the file:
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@@
 	)
 	(no_connect
+		(at 276.86 106.68)
+	)
+	(no_connect
+		(at 276.86 109.22)
+	)
+	(no_connect
+		(at 231.14 73.66)
+	)
+	(no_connect
+		(at 220.98 106.68)
+	)
+	(no_connect
+		(at 205.74 45.72)
+	)
+	(no_connect
+		(at 276.86 101.6)
+	)
+	(no_connect
 		(at 25.4 48.26)
 	)
 	(no_connect
+		(at 276.86 104.14)
+	)
+	(no_connect
+		(at 231.14 68.58)
+	)
+	(no_connect
+		(at 231.14 66.04)
+	)
+	(no_connect
+		(at 231.14 71.12)
+	)
+	(no_connect
 		(at 25.4 45.72)
 	)
@@
 	)
 	(no_connect
+		(at 120.65 55.88)
+	)
+	(no_connect
+		(at 231.14 76.2)
+	)
+	(no_connect
+		(at 205.74 35.56)
+	)
+	(no_connect
+		(at 120.65 53.34)
+	)
+	(no_connect
 		(at 25.4 55.88)
 	)
@@
 	)
 	(no_connect
+		(at 220.98 101.6)
+	)
+	(no_connect
 		(at 60.96 45.72)
 	)
 	(no_connect
+		(at 205.74 43.18)
+	)
+	(no_connect
+		(at 205.74 48.26)
+	)
+	(no_connect
+		(at 220.98 99.06)
+	)
+	(no_connect
 		(at 25.4 58.42)
 	)
@@
 	)
 	(no_connect
+		(at 231.14 78.74)
+	)
+	(no_connect
 		(at 60.96 48.26)
 	)
+	(no_connect
+		(at 220.98 104.14)
+	)
+	(no_connect
+		(at 205.74 38.1)
+	)
 	(bus_entry
 		(at 182.88 109.22)
@@
 		)
 	)
-	(hierarchical_label "{DATA_BUS}"
+	(hierarchical_label "d[0..7]"
 		(shape bidirectional)
 		(at 214.63 135.89 0)
@@
 		)
 	)
-	(hierarchical_label "{DATA_BUS}"
+	(hierarchical_label "d[0..7]"
 		(shape bidirectional)
 		(at 119.38 101.6 0)
@@
 		)
 	)
-	(hierarchical_label "{DATA_BUS}"
+	(hierarchical_label "d[0..7]"
 		(shape bidirectional)
 		(at 165.1 109.22 270)
@@
 		)
 	)
-	(hierarchical_label "{ADDRESS_BUS}"
+	(hierarchical_label "addr[0..19]"
 		(shape bidirectional)
 		(at 77.47 24.13 0)
@@
 		)
 	)
-	(hierarchical_label "{ADDRESS_BUS}"
+	(hierarchical_label "addr[0..19]"
 		(shape bidirectional)
 		(at 180.34 100.33 0)
@@
 		)
 	)
-	(hierarchical_label "{ADDRESS_BUS}"
+	(hierarchical_label "addr[0..19]"
 		(shape bidirectional)
 		(at 214.63 87.63 0)
