File: power.kicad_sch (KiCad schematic)
At the start: 4 parts, among them J1 ATX-20, J2 F_PANEL, Q1 2N7000, U4 CD74HCT74E

Commit message: power delivery to compute basics
Signed-off-by: Lucy Mielke <user@domain.tld>
Parts:
- added C6, C7: 0.1uF, Capacitor_THT:C_Disc_D3.0mm_W1.6mm_P2.50mm, symbol Device:C
- added R2, R3: 10k, Resistor_THT:R_Axial_DIN0204_L3.6mm_D1.6mm_P5.08mm_Horizontal, symbol Device:R
- added U5: SN74HCT08N, SN74HCT08N AND-Gate IC:DIP794W45P254L1969H508Q14, symbol SN74HCT08N:SN74HCT08N
Connections:
- net 5V: now also C7.1, R2.1, U5.14 (VCC)
- net 5VSB: now also U4.1 (1~R), U4.4 (1~S), C6.2, R3.1
- net GND: now also U4.10 (2~S), U4.11 (2CP), U4.13 (2~R), U4.8 (2~Q), U4.9 (2Q), C6.1, C7.2, U5.10 (3B), U5.12 (4A), U5.13 (4B), U5.4 (2A), U5.5 (2B), U5.7 (GND), U5.9 (3A)
- net PWR_BTN: now also R3.2
- net PWR_OK: now also U5.1 (1A)
- net at U4.2 (1D): now also U4.6 (1~Q)
- new net: R2.2, U5.2 (1B)
- new net RSTBTN: U5.3 (1Y)
- no-connect marks 3 -> 7
Other:
- note added: "AND-gate, that uses the power-OK signal and 5V to send a reset-signal to the intel clock IC for power-on reset"
- note added: "Flip-Flop circuit that turns on the PSU, using the 5V stand-by power to operate"
- moved on the sheet: J2, Q1, U4

Commit message: Complete UART connection
Signed-off-by: Lucy Mielke <user@domain.tld>
Connections:
- net GND: no longer U5.4 (2A), U5.5 (2B)
- net IO_G2A: now reaches U5.6 (2Y)
- new net IORC: U5.4 (2A)
- new net IOWC: U5.5 (2B)
- no-connect marks 7 -> 6
Other:
- note added: "AND-gate 1 uses the power-OK signal and 5V to send a reset-signal to the intel clock IC for power-on reset AND-Gate 2 controls the enable signal for the IO controller using 8288 IO signals"
- note removed: "AND-gate, that uses the power-OK signal and 5V to send a reset-signal to the intel clock IC for power-on reset"
Changed lines of the file:
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@@
 		(comment 1 "${COMMENT1}")
 	)
-	(text "AND-gate, that uses\nthe power-OK signal and 5V\nto send a reset-signal to the\nintel clock IC for power-on reset"
+	(text "AND-gate 1 uses\nthe power-OK signal and 5V\nto send a reset-signal to the\nintel clock IC for power-on reset\n\nAND-Gate 2 controls the enable signal\nfor the IO controller using\n8288 IO signals"
 		(exclude_from_sim no)
-		(at 111.76 28.194 0)
+		(at 104.902 24.638 0)
 		(effects
 			(font
@@
 	)
 	(junction
-		(at 93.98 54.61)
-		(diameter 0)
-		(color 0 0 0 0)
-	)
-	(junction
 		(at 38.1 162.56)
 		(diameter 0)
@@
 	(junction
 		(at 93.98 62.23)
-		(diameter 0)
-		(color 0 0 0 0)
-	)
-	(junction
-		(at 93.98 57.15)
 		(diameter 0)
 		(color 0 0 0 0)
@@
 	)
 	(no_connect
-		(at 132.08 49.53)
-	)
-	(no_connect
 		(at 132.08 54.61)
 	)
@@
 	(wire
 		(pts
-			(xy 93.98 54.61) (xy 93.98 57.15)
-		)
-		(stroke
-			(width 0)
-			(type default)
-		)
-	)
-	(wire
-		(pts
 			(xy 24.13 124.46) (xy 24.13 132.08)
 		)
@@
 	(wire
 		(pts
+			(xy 137.16 49.53) (xy 132.08 49.53)
+		)
+		(stroke
+			(width 0)
+			(type default)
+		)
+	)
+	(wire
+		(pts
 			(xy 43.18 72.39) (xy 43.18 78.74)
 		)
@@
 	(wire
 		(pts
-			(xy 93.98 52.07) (xy 93.98 54.61)
-		)
-		(stroke
-			(width 0)
-			(type default)
-		)
-	)
-	(wire
-		(pts
 			(xy 16.51 69.85) (xy 16.51 73.66)
 		)
@@
 	(wire
 		(pts
-			(xy 93.98 54.61) (xy 96.52 54.61)
-		)
-		(stroke
-			(width 0)
-			(type default)
-		)
-	)
-	(wire
-		(pts
 			(xy 133.35 27.94) (xy 133.35 34.29)
 		)
@@
 	(wire
 		(pts
-			(xy 96.52 52.07) (xy 93.98 52.07)
-		)
-		(stroke
-			(width 0)
-			(type default)
-		)
-	)
-	(wire
-		(pts
 			(xy 25.4 69.85) (xy 16.51 69.85)
 		)
@@
 	(wire
 		(pts
+			(xy 90.17 52.07) (xy 96.52 52.07)
+		)
+		(stroke
+			(width 0)
+			(type default)
+		)
+	)
+	(wire
+		(pts
 			(xy 38.1 72.39) (xy 43.18 72.39)
 		)
@@
 		(pts
 			(xy 24.13 116.84) (xy 24.13 113.03)
+		)
+		(stroke
+			(width 0)
+			(type default)
+		)
+	)
+	(wire
+		(pts
+			(xy 90.17 54.61) (xy 96.52 54.61)
 		)
 		(stroke
@@
 		)
 	)
+	(hierarchical_label "IO_G2A"
+		(shape input)
+		(at 137.16 49.53 0)
+		(effects
+			(font
+				(size 1.27 1.27)
+			)
+			(justify left)
+		)
+	)
 	(hierarchical_label "PS_ON"
 		(shape input)
@@
 		(shape input)
 		(at 21.59 22.86 180)
+		(effects
+			(font
+				(size 1.27 1.27)
+			)
+			(justify right)
+		)
+	)
+	(hierarchical_label "IOWC"
+		(shape input)
+		(at 90.17 54.61 180)
 		(effects
 			(font
@@
 		)
 	)
+	(hierarchical_label "IORC"
+		(shape input)
+		(at 90.17 52.07 180)
+		(effects
+			(font
+				(size 1.27 1.27)
+			)
+			(justify right)
+		)
+	)

Commit message: reorganise
Signed-off-by: Lucy Mielke <user@domain.tld>
Other:
- note added: "Power"
- moved on the sheet: C6, C7, J1, J2, Q1, R2, R3, U4, U5

Commit message: IDE controller/connector
Signed-off-by: Lucy Mielke <user@domain.tld>
Parts:
- added R27: 3,3R, Resistor_THT:R_Axial_DIN0204_L3.6mm_D1.6mm_P5.08mm_Horizontal, symbol Device:R
Connections:
- net 5V: now also R27.1
- net GND: no longer U5.10 (3B), U5.9 (3A)
- net HDD_LED+: now also R27.2
- net IORC: now also U5.10 (3B)
- net IDE_LE: now reaches U5.8 (3Y)
- new net IDE_CS: U5.9 (3A)
- no-connect marks 6 -> 5
Changed lines of the file:
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@@
+	)
+	(junction
+		(at 36.83 71.12)
+		(diameter 0)
+		(color 0 0 0 0)
 	)
 	(junction
@@
 	)
 	(junction
-		(at 214.63 76.2)
-		(diameter 0)
-		(color 0 0 0 0)
-	)
-	(junction
 		(at 214.63 81.28)
 		(diameter 0)
@@
 		(color 0 0 0 0)
 	)
-	(junction
-		(at 214.63 78.74)
-		(diameter 0)
-		(color 0 0 0 0)
-	)
 	(no_connect
 		(at 43.18 81.28)
 	)
 	(no_connect
-		(at 252.73 68.58)
-	)
-	(no_connect
 		(at 55.88 81.28)
 	)
@@
 	(wire
 		(pts
-			(xy 214.63 73.66) (xy 217.17 73.66)
-		)
-		(stroke
-			(width 0)
-			(type default)
-		)
-	)
-	(wire
-		(pts
 			(xy 83.82 128.27) (xy 83.82 135.89)
 		)
@@
 	(wire
 		(pts
-			(xy 214.63 76.2) (xy 214.63 78.74)
-		)
-		(stroke
-			(width 0)
-			(type default)
-		)
-	)
-	(wire
-		(pts
 			(xy 34.29 76.2) (xy 34.29 80.01)
 		)
@@
 	(wire
 		(pts
+			(xy 36.83 71.12) (xy 43.18 71.12)
+		)
+		(stroke
+			(width 0)
+			(type default)
+		)
+	)
+	(wire
+		(pts
 			(xy 97.79 146.05) (xy 97.79 153.67)
 		)
@@
 	(wire
 		(pts
-			(xy 214.63 73.66) (xy 214.63 76.2)
+			(xy 31.75 71.12) (xy 36.83 71.12)
 		)
 		(stroke
@@
 	(wire
 		(pts
-			(xy 214.63 76.2) (xy 217.17 76.2)
+			(xy 213.36 73.66) (xy 217.17 73.66)
 		)
 		(stroke
@@
 		)
 	)
-	(label "HDD_LED+"
-		(at 43.18 71.12 180)
-		(effects
-			(font
-				(size 1.27 1.27)
-			)
-			(justify right bottom)
-		)
-	)
-	(label "HDD_LED-"
-		(at 43.18 73.66 180)
-		(effects
-			(font
-				(size 1.27 1.27)
-			)
-			(justify right bottom)
-		)
-	)
 	(label "PLED+"
 		(at 55.88 71.12 0)
@@
 			)
 			(justify left)
+		)
+	)
+	(hierarchical_label "HDD_LED-"
+		(shape passive)
+		(at 43.18 73.66 180)
+		(effects
+			(font
+				(size 1.27 1.27)
+			)
+			(justify right)
 		)
 	)
@@
 		)
 	)
+	(hierarchical_label "5V"
+		(shape input)
+		(at 36.83 63.5 90)
+		(effects
+			(font
+				(size 1.27 1.27)
+			)
+			(justify left)
+		)
+	)
+	(hierarchical_label "IDE_LE"
+		(shape output)
+		(at 252.73 68.58 0)
+		(effects
+			(font
+				(size 1.27 1.27)
+			)
+			(justify left)
+		)
+	)
 	(hierarchical_label "3.3V"
 		(shape output)
@@
 			)
 			(justify left)
+		)
+	)
+	(hierarchical_label "IORC"
+		(shape input)
+		(at 217.17 76.2 180)
+		(effects
+			(font
+				(size 1.27 1.27)
+			)
+			(justify right)
+		)
+	)
+	(hierarchical_label "IDE_CS"
+		(shape input)
+		(at 213.36 73.66 180)
+		(effects
+			(font
+				(size 1.27 1.27)
+			)
+			(justify right)
+		)
+	)
+	(hierarchical_label "HDD_LED+"
+		(shape passive)
+		(at 31.75 71.12 180)
+		(effects
+			(font
+				(size 1.27 1.27)
+			)
+			(justify right)
 		)
 	)
@@
 					(unit 1)
 				)
+			)
+		)
+	)
+	(symbol
+		(lib_id "Device:R")
+		(at 36.83 67.31 0)
+		(unit 1)
+		(body_style 1)
+		(exclude_from_sim no)
+		(in_bom yes)
+		(on_board yes)
+		(in_pos_files yes)
+		(dnp no)
+		(fields_autoplaced yes)
+		(property "Reference" "R27"
+			(at 39.37 66.0399 0)
+			(show_name no)
+			(do_not_autoplace no)
+			(effects
+				(font
+					(size 1.27 1.27)
+				)
+				(justify left)
+			)
+		)
+		(property "Value" "3,3R"
+			(at 39.37 68.5799 0)
+			(show_name no)
+			(do_not_autoplace no)
+			(effects
+				(font
+					(size 1.27 1.27)
+				)
+				(justify left)
+			)
+		)
+		(property "Footprint" "Resistor_THT:R_Axial_DIN0204_L3.6mm_D1.6mm_P5.08mm_Horizontal"
+			(at 35.052 67.31 90)
+			(hide yes)
+			(show_name no)
+			(do_not_autoplace no)
+			(effects
+				(font
+					(size 1.27 1.27)
+				)
+			)
+		)
+		(property "Datasheet" ""
+			(at 36.83 67.31 0)
+			(hide yes)
+			(show_name no)
+			(do_not_autoplace no)
+			(effects
+				(font
+					(size 1.27 1.27)
+				)
+			)
+		)
+		(property "Description" "Resistor"
+			(at 36.83 67.31 0)
+			(hide yes)
+			(show_name no)
+			(do_not_autoplace no)
+			(effects
+				(font
+					(size 1.27 1.27)
+				)
+			)
+		)
+		(pin "2"
+		)
+		(pin "1"
+		)
+		(instances
+			(project "scarlet-8088"
+				(path "/6bf7a8bc-eb70-43f6-b16b-1b538dd0d96d/5b0a69b8-537a-4e54-9053-3d6e1d6f1e22"
+					(reference "R27")
+					(unit 1)
+				)

Commit message: Fix ERC errors
Signed-off-by: Lucy Mielke <user@domain.tld>
Connections:
- net GND: no longer U4.8 (2~Q), U4.9 (2Q)
- no-connect marks 5 -> 10
Changed lines of the file:
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@@
-	)
-	(junction
-		(at 135.89 140.97)
-		(diameter 0)
-		(color 0 0 0 0)
 	)
 	(junction
@@
 	)
 	(no_connect
+		(at 135.89 140.97)
+	)
+	(no_connect
 		(at 55.88 81.28)
+	)
+	(no_connect
+		(at 55.88 73.66)
+	)
+	(no_connect
+		(at 43.18 78.74)
+	)
+	(no_connect
+		(at 135.89 138.43)
 	)
 	(no_connect
@@
 		(at 252.73 71.12)
 	)
+	(no_connect
+		(at 55.88 71.12)
+	)
 	(wire
 		(pts
@@
 	(wire
 		(pts
-			(xy 135.89 140.97) (xy 135.89 168.91)
-		)
-		(stroke
-			(width 0)
-			(type default)
-		)
-	)
-	(wire
-		(pts
 			(xy 100.33 130.81) (xy 97.79 130.81)
 		)
@@
 		(pts
 			(xy 34.29 76.2) (xy 34.29 80.01)
-		)
-		(stroke
-			(width 0)
-			(type default)
-		)
-	)
-	(wire
-		(pts
-			(xy 135.89 138.43) (xy 135.89 140.97)
 		)
 		(stroke
@@
 					(unit 1)
 				)
-			)
-		)
-	)
-	(symbol
-		(lib_id "power:GND")
-		(at 135.89 168.91 0)
-		(unit 1)
-		(body_style 1)
-		(exclude_from_sim no)
-		(in_bom yes)
-		(on_board yes)
-		(in_pos_files yes)
-		(dnp no)
-		(fields_autoplaced yes)
-		(property "Reference" "#PWR019"
-			(at 135.89 175.26 0)
-			(hide yes)
-			(show_name no)
-			(do_not_autoplace no)
-			(effects
-				(font
-					(size 1.27 1.27)
-				)
-			)
-		)
-		(property "Value" "GND"
-			(at 135.89 173.99 0)
-			(show_name no)
-			(do_not_autoplace no)
-			(effects
-				(font
-					(size 1.27 1.27)
-				)
-			)
-		)
-		(property "Footprint" ""
-			(at 135.89 168.91 0)
-			(hide yes)
-			(show_name no)
-			(do_not_autoplace no)
-			(effects
-				(font
-					(size 1.27 1.27)
-				)
-			)
-		)
-		(property "Datasheet" ""
-			(at 135.89 168.91 0)
-			(hide yes)
-			(show_name no)
-			(do_not_autoplace no)
-			(effects
-				(font
-					(size 1.27 1.27)
-				)
-			)
-		)
-		(property "Description" "Power symbol creates a global label with name \"GND\" , ground"
-			(at 135.89 168.91 0)
-			(hide yes)
-			(show_name no)
-			(do_not_autoplace no)
-			(effects
-				(font
-					(size 1.27 1.27)
-				)
-			)
-		)
-		(pin "1"
-		)
-		(instances
-			(project "scarlet-8088"
-				(path "/6bf7a8bc-eb70-43f6-b16b-1b538dd0d96d/5b0a69b8-537a-4e54-9053-3d6e1d6f1e22"
-					(reference "#PWR019")
-					(unit 1)
-				)
