File: io.kicad_sch (KiCad schematic)
At the start: 9 parts, among them SW1 SW_DIP_x08, U12 8255A, U13 SN74HCT138N, U23 8259A

Commit message: change Mini-DIN-6 Footprint; Place ISA slots correctly
Signed-off-by: Lucy Mielke <user@domain.tld>
Parts:
- SW1: footprint Button_Switch_THT:SW_DIP_SPSTx02_Piano_10.8x6.64mm_W7.62mm_P2.54mm -> Button_Switch_THT:SW_DIP_SPSTx08_Piano_10.8x21.88mm_W7.62mm_P2.54mm
Changed lines of the file:
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@@
 			)
 		)
-		(property "Footprint" "Button_Switch_THT:SW_DIP_SPSTx02_Piano_10.8x6.64mm_W7.62mm_P2.54mm"
+		(property "Footprint" "Button_Switch_THT:SW_DIP_SPSTx08_Piano_10.8x21.88mm_W7.62mm_P2.54mm"
 			(at 172.72 46.99 0)
 			(hide yes)
