File: io_ps2.kicad_sch (KiCad schematic)
At the start: 19 parts, among them J4 Mini-DIN-6 KBD, J5 Mini-DIN-6 Mouse, U25 Intel 8242, Y3 12MHz

Commit message: Added compatible RJ45 Ethernet
Signed-off-by: Lucy Mielke <user@domain.tld>
Other:
- note added: "PS/2 Mouse and Keyboard"
Changed lines of the file:
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@@
 		(comment 1 "${COMMENT1}")
+	)
+	(text "PS/2 Mouse and Keyboard"
+		(exclude_from_sim no)
+		(at 138.684 19.558 0)
+		(effects
+			(font
+				(size 1.905 1.905)
+			)
+		)
 	)
 	(junction

Commit message: Fix ERC errors
Signed-off-by: Lucy Mielke <user@domain.tld>
Changed lines of the file:
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@@
 		)
 	)
-	(hierarchical_label "{ADDRESS_BUS}"
+	(hierarchical_label "addr[0..19]"
 		(shape bidirectional)
 		(at 63.5 66.04 180)
@@
 		)
 	)
-	(hierarchical_label "{DATA_BUS}"
+	(hierarchical_label "d[0..7]"
 		(shape bidirectional)
 		(at 66.04 96.52 180)

Commit message: change Mini-DIN-6 Footprint; Place ISA slots correctly
Signed-off-by: Lucy Mielke <user@domain.tld>
Parts:
- J4, J5: footprint Connector_DIN:DIN41612_M-invers_3x2+10_Female_Horizontal_THT -> minidin_6_ps2_pcb_mount:minidin_6_ps2_pcb_mount
Changed lines of the file:
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@@
 			)
 		)
-		(property "Footprint" "Connector_DIN:DIN41612_M-invers_3x2+10_Female_Horizontal_THT"
+		(property "Footprint" "minidin_6_ps2_pcb_mount:minidin_6_ps2_pcb_mount"
 			(at 167.64 49.53 0)
 			(hide yes)
@@
 			)
 		)
-		(property "Footprint" "Connector_DIN:DIN41612_M-invers_3x2+10_Female_Horizontal_THT"
+		(property "Footprint" "minidin_6_ps2_pcb_mount:minidin_6_ps2_pcb_mount"
 			(at 167.64 73.66 0)
 			(hide yes)
