File: scarlet-8088.kicad_pcb (KiCad board)
At the start: 4 copper layers, 305 x 244 mm, 140 parts, among them J1 ATX-20, J10 Bus_ISA_8bit, J2 F_PANEL, J3 DE-9SA-J4-2R, J4 Mini-DIN-6 KBD, J5 Mini-DIN-6 Mouse, J6 RJ45_Amphenol_RJMG1BD3B8K1ANR, J7 Conn_02x20_Odd_Even, J8 Bus_ISA_8bit, J9 Bus_ISA_8bit, Q1 2N7000, SW1 SW_DIP_x08, U1 Intel_8088, U10 AS6C4008-55PCN, U11 74HCT373, U12 8255A, U13 SN74HCT138N, U14 SN74HCT245N, U15 AS6C4008-55PCN, U16 28C256, U17 CD74HCT14E, U18 CD74HCT10E, U19 TL16C550BN, U2 8087, U20 CD74HCT30E, U21 MAX232, U22 MAX232, U23 8259A, U24 8254, U25 Intel 8242, U26 Realtek RTL8019AS, U27 93LCxxC, U28 74HCT688 (CD74HCT688E), U29 SN74HCT245N, U3 8284, U30 SN74HCT245N, U31 SN74HCT573N, U32 SN74HCT32N, U33 L7905, U4 CD74HCT74E, U5 SN74HCT08N, U6 8288, U7 SN74HCT138N, U8 SN74HCT08N, U9 CD74HCT21E, Y1 14.31818 MHz, Y2 1.8432MHZ, Y3 12MHz

Commit message: Reset footprint placement; place Power System footprints
Signed-off-by: Lucy Mielke <user@domain.tld>
Parts:
- moved U33 844.5 mm to (-87.4, 1048.7)
- moved C54 835.9 mm to (-77.5, 1046.3)
- moved C53 822.0 mm to (-73.3, 1039.9)
- moved C52 821.5 mm to (-84.8, 1039.9)
- moved U27 811.3 mm to (-74.2, 848.1)
- moved C44 807.0 mm to (-62.9, 843.1)
- moved C43 793.7 mm to (-57.3, 843.1)
- moved U26 790.4 mm to (-63.6, 828.6)
- moved R22 787.4 mm to (-63.0, 840.0)
- moved U28 759.7 mm to (-96.7, 977.5)
- moved R25 753.8 mm to (-57.6, 965.4)
- moved C50 738.8 mm to (-51.3, 962.4)
- moved U30 733.1 mm to (-95.9, 966.3)
- moved C47 731.6 mm to (-57.6, 959.9)
- moved U31 730.0 mm to (-56.8, 952.9)
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Routing:
- added copper zone on In2.Cu, net /5V
- added copper zone on B.Cu, net GND
- added copper zone on F.Cu, net GND
- added copper zone on In1.Cu, net GND
