File: scarlet-8088.kicad_pcb (KiCad board)
At the start: 4 copper layers, 305 x 244 mm, 140 parts, among them J1 ATX-20, J10 Bus_ISA_8bit, J2 F_PANEL, J3 DE-9SA-J4-2R, J4 Mini-DIN-6 KBD, J5 Mini-DIN-6 Mouse, J6 RJ45_Amphenol_RJMG1BD3B8K1ANR, J7 Conn_02x20_Odd_Even, J8 Bus_ISA_8bit, J9 Bus_ISA_8bit, Q1 2N7000, SW1 SW_DIP_x08, U1 Intel_8088, U10 AS6C4008-55PCN, U11 74HCT373, U12 8255A, U13 SN74HCT138N, U14 SN74HCT245N, U15 AS6C4008-55PCN, U16 28C256, U17 CD74HCT14E, U18 CD74HCT10E, U19 TL16C550BN, U2 8087, U20 CD74HCT30E, U21 MAX232, U22 MAX232, U23 8259A, U24 8254, U25 Intel 8242, U26 Realtek RTL8019AS, U27 93LCxxC, U28 74HCT688 (CD74HCT688E), U29 SN74HCT245N, U3 8284, U30 SN74HCT245N, U31 SN74HCT573N, U32 SN74HCT32N, U33 L7905, U4 CD74HCT74E, U5 SN74HCT08N, U6 8288, U7 SN74HCT138N, U8 SN74HCT08N, U9 CD74HCT21E, Y1 14.31818 MHz, Y2 1.8432MHZ, Y3 12MHz

Commit message: place compute block
Signed-off-by: Lucy Mielke <user@domain.tld>
Parts:
- moved R1 424.9 mm to (378.0, 215.0)
- moved Q1 424.1 mm to (-46.1, 220.2)
- moved U1 419.5 mm to (348.0, 214.8), turned to -90 degrees
- moved R3 414.8 mm to (-49.6, 218.5)
- moved C6 412.2 mm to (-40.0, 218.5)
- moved U2 407.3 mm to (355.2, 197.2)
- moved U4 407.2 mm to (-53.3, 215.6)
- moved C4 400.3 mm to (328.4, 256.5), turned to 0 degrees
- moved C5 399.8 mm to (331.1, 251.5), turned to 180 degrees
- moved C2 389.0 mm to (368.4, 194.5)
- moved C1 367.4 mm to (350.7, 228.0), turned to -90 degrees
- moved U3 363.2 mm to (348.6, 254.9)
- moved C3 356.4 mm to (343.0, 257.6)
- moved Y1 355.8 mm to (335.0, 251.5)
- moved R4 314.9 mm to (248.4, 194.3), turned to -90 degrees
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
Commit message: Component placement fully redone
Signed-off-by: Lucy Mielke <user@domain.tld>
Parts:
- moved U33 983.2 mm to (238.3, 121.0), turned to -90 degrees
- moved C52 974.4 mm to (225.0, 116.1), turned to 0 degrees
- moved C53 960.1 mm to (225.1, 127.4), turned to 0 degrees
- moved C54 959.5 mm to (227.5, 136.6), turned to 180 degrees
- moved R26 815.6 mm to (358.8, 262.3), turned to 180 degrees
- moved U28 809.1 mm to (273.0, 257.7)
- moved U27 808.6 mm to (355.0, 162.9)
- moved C48 808.1 mm to (327.3, 263.0)
- moved C44 803.9 mm to (352.3, 154.8)
- moved C43 803.6 mm to (373.1, 164.5), turned to 0 degrees
- moved R25 803.6 mm to (293.2, 242.5)
- moved U29 798.4 mm to (301.0, 263.0)
- moved U32 793.1 mm to (340.0, 287.0)
- moved C51 784.5 mm to (336.2, 298.2)
- moved U26 782.5 mm to (366.7, 175.1)
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
Commit message: use more of the available space for the placement
Signed-off-by: Lucy Mielke <user@domain.tld>
Parts:
- moved U18 180.2 mm to (258.8, 331.2), turned to 0 degrees
- moved C11 174.6 mm to (273.7, 324.8), turned to 180 degrees
- moved U30 155.0 mm to (234.7, 161.9), turned to 180 degrees
- moved C9 153.2 mm to (253.7, 312.3), turned to 180 degrees
- moved U9 150.6 mm to (271.1, 306.0), turned to 180 degrees
- moved C19 150.5 mm to (253.7, 310.2), turned to 180 degrees
- moved C49 148.2 mm to (234.8, 188.2), turned to 0 degrees
- moved U17 147.7 mm to (283.3, 288.6), turned to 90 degrees
- moved U28 141.5 mm to (273.6, 116.2), turned to 0 degrees
- moved C51 138.9 mm to (236.9, 201.1), turned to -90 degrees
- moved U7 137.7 mm to (254.9, 299.0), turned to 180 degrees
- moved C47 136.6 mm to (281.6, 113.5), turned to 180 degrees
- moved C18 133.0 mm to (270.6, 286.5), turned to 180 degrees
- moved C50 127.3 mm to (252.4, 187.6), turned to 0 degrees
- moved U31 125.7 mm to (256.2, 173.5), turned to 180 degrees
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