File: scarlet-8088.kicad_pcb (KiCad board)
At the start: 4 copper layers, 305 x 244 mm, 140 parts, among them J1 ATX-20, J10 Bus_ISA_8bit, J2 F_PANEL, J3 DE-9SA-J4-2R, J4 Mini-DIN-6 KBD, J5 Mini-DIN-6 Mouse, J6 RJ45_Amphenol_RJMG1BD3B8K1ANR, J7 Conn_02x20_Odd_Even, J8 Bus_ISA_8bit, J9 Bus_ISA_8bit, Q1 2N7000, SW1 SW_DIP_x08, U1 Intel_8088, U10 AS6C4008-55PCN, U11 74HCT373, U12 8255A, U13 SN74HCT138N, U14 SN74HCT245N, U15 AS6C4008-55PCN, U16 28C256, U17 CD74HCT14E, U18 CD74HCT10E, U19 TL16C550BN, U2 8087, U20 CD74HCT30E, U21 MAX232, U22 MAX232, U23 8259A, U24 8254, U25 Intel 8242, U26 Realtek RTL8019AS, U27 93LCxxC, U28 74HCT688 (CD74HCT688E), U29 SN74HCT245N, U3 8284, U30 SN74HCT245N, U31 SN74HCT573N, U32 SN74HCT32N, U33 L7905, U4 CD74HCT74E, U5 SN74HCT08N, U6 8288, U7 SN74HCT138N, U8 SN74HCT08N, U9 CD74HCT21E, Y1 14.31818 MHz, Y2 1.8432MHZ, Y3 12MHz

Commit message: Routing rev1.0 finished
Signed-off-by: Lucy Mielke <user@domain.tld>
Routing:
- net /Compute/addr6: track 643.5 -> 496.2 mm, vias 22 -> 30
- net /Compute/addr4: track 571.6 -> 476.2 mm, vias 21 -> 28
- net /Compute/d5: track 752.9 -> 658.3 mm, vias 38 -> 36
- net /Compute/d6: track 762.2 -> 668.5 mm, vias 35 -> 51
- net /Compute/addr2: track 653.3 -> 568.0 mm, vias 24 -> 39
- net /Compute/addr3: track 553.1 -> 485.7 mm, vias 25 -> 29
- net /IO/IDE/IDE_D11: track 100.0 -> 45.2 mm
- net /Compute/d7: track 686.3 -> 738.9 mm, vias 32 -> 51
- net /Compute/addr12: track 600.0 -> 547.8 mm, vias 20 -> 32
- net /MRDC: track 606.0 -> 554.0 mm, vias 26 -> 35
- net /Compute/d0: track 738.7 -> 686.9 mm, vias 32 -> 43
- net /IO/IDE/IDE_D13: track 93.7 -> 45.5 mm
- net /RSTBTN_INV: track 389.7 -> 342.0 mm, vias 16 -> 19
- net /Compute/addr13: track 563.2 -> 515.7 mm, vias 24 -> 22
- net /Compute/d2: track 672.9 -> 719.9 mm, vias 32 -> 41
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- added copper zone on F.Cu, net /5V
- added copper zone on In1.Cu, net /5V
- removed copper zone on B.Cu, net GND
